File: CompactBeamspring/CompactBeamspring.kicad_pcb (KiCad board)
At the start: 2 copper layers, 163.6 x 18.8 mm, 34 parts, among them J1 BEAMSPRING CONNECTOR, J2 PadsToShort, J3 EXPANSION HEADER, U1 MCP4921-E, U2 LM339A, U3 74AHC595, U4 74AHC595, U5 ProMicro, U7 74AHC595

Commit message: Updated to rev. 1.4
Parts:
- removed NT1: Net-Tie_3, NetTie:NetTie-3_THT_Pad0.3mm
- removed REF** (x2): tooling_hole, TH-XWhatsIt:tooling_hole
- added H2: ToolingHole, TH-XWhatsIt:tooling_hole, F.Cu at (76.7, 156.4)
- added H3: ToolingHole, TH-XWhatsIt:tooling_hole, F.Cu at (250.9, 158.8)
- added J4: Conn_02x05_Odd_Even, Connector_PinHeader_2.54mm:PinHeader_2x05_P2.54mm_Vertical, F.Cu at (110.4, 146.4)
- moved J2 17.8 mm to (80.5, 147.0)
- moved NT2 17.8 mm to (83.2, 145.9)
- moved R6 17.8 mm to (103.8, 147.4)
- moved R7 17.8 mm to (103.8, 149.4)
- moved R8 17.8 mm to (103.8, 151.4)
- moved U5 17.8 mm to (90.7, 151.3)
Connections:
- net HEADER1 renamed HEADER1_LED5
- net HEADER2 renamed HEADER2_LED4
- net Net-(R6-Pad2) renamed BUTTON1
- net Net-(R8-Pad1) renamed BUTTON2
- C1 pad 1: GNDA -> GND
- C2 pad 1: GNDD -> GND
- C3 pad 1: GNDA -> GND
- C4 pad 1: GNDD -> GND
- C5 pad 1: GNDD -> GND
- C6 pad 1: GNDA -> GND
- H1 pad 1: GNDA -> GND
- J1 pad 30: GNDD -> GND
- J1 pad 5: GNDD -> GND
- J3 pad 6: GNDD -> GND
- R2 pad 1: GNDA -> GND
- R5 pad 1: GNDA -> GND
- R7 pad 2: GNDD -> GND
- R8 pad 2: GNDD -> GND
- U1 pad 5: GNDA -> GND
- U1 pad 7: GNDA -> GND
- U2 pad 12: GNDA -> GND
- U3 pad 13: GNDD -> GND
- U3 pad 8: GNDD -> GND
- U4 pad 13: GNDD -> GND
- U4 pad 8: GNDD -> GND
- U5 pad 11: Net-(U5-Pad11) -> LED2
- U5 pad 12: Net-(U5-Pad12) -> LED3
- U5 pad 19: Net-(U5-Pad19) -> LED1
- U5 pad 20: Net-(U5-Pad20) -> BUTTON3
- U7 pad 13: GNDD -> GND
- U7 pad 8: GNDD -> GND
Routing:
- net GND: track 22.2 -> 273.3 mm, vias 0 -> 241
- net GNDA: track 131.3 -> 0.00 mm, vias 30 -> 0
- net GNDD: track 110.9 -> 0.00 mm, vias 73 -> 0
- net BUTTON3: track 0.00 -> 35.1 mm
- net HEADER3: track 46.3 -> 76.2 mm
- net HEADER2_LED4: track 34.7 -> 64.3 mm, vias 2 -> 1
- net HEADER4: track 44.9 -> 74.0 mm
- net HEADER1_LED5: track 45.2 -> 70.0 mm, vias 2 -> 1
- net LED1: track 0.00 -> 22.6 mm
- net LED3: track 0.00 -> 22.2 mm, vias 0 -> 1
- net LED2: track 0.00 -> 21.7 mm, vias 0 -> 1
- net +5VD: track 161.2 -> 181.3 mm
- net BUTTON2: track 15.1 -> 35.2 mm
- net CLOCK: track 126.5 -> 146.5 mm
- net LOADCOL: track 122.5 -> 142.2 mm
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- added copper zone on B.Cu, net GND
- added copper zone on F.Cu, net GND
- removed copper zone on B.Cu, net GNDA
- removed copper zone on F.Cu, net GNDA
- removed copper zone on B.Cu, net GNDD
- removed copper zone on F.Cu, net GNDD
Other:
- board size 163.6 x 18.8 mm -> 181.3 x 18.9 mm
- board text added: "+5V"
- board text added: "< Left side of keyboard"
- board text added: "BTNs"
- board text added: "Beamspring"
- board text added: "Compact-"
- board text added: "Compact-Beamspring Rev1.4"
- board text added: "EN"
- board text added: "Expansion Header e.g. Solenoid Drv."
- board text added: "LEDs no res"
- board text added: "Left side of > keyboard"
- board text added: "More Expansion e.g. 3278 extra leds+buttons"
- board text added: "Mount ProMicro and 90-degree pinheaders on this side"
- board text added: "Rev1.4"
- board text added: "TRIG"
- board text removed: "Compact-Beamspring Rev1.3"
